Commit message: add ros2_control

File: description/depth_camera.xacro (robot description, xacro)
@@ -4,5 +4,5 @@
         <parent link="chassis"/>
         <child link="camera_link"/>
-        <origin xyz="0.340 0 0.069" rpy="0 0.18 0"/>
+        <origin xyz="0.305 0 0.08" rpy="0 0 0"/>
     </joint>
     <link name="camera_link">
@@ -21,24 +21,45 @@
     <link name="camera_link_optical"></link>
     <gazebo reference="camera_link">
-        <material>Gazebo/Black</material>
-        <sensor name="camera" type="depth">
-            <pose> 0 0 0 0 0 0 </pose>
-            <visualize>true</visualize>
-            <update_rate>10</update_rate>
-            <camera>
-                <camera_info_topic>camera/camera_info</camera_info_topic>
-                <horizontal_fov>1.089</horizontal_fov>
-                <image>
-                    <format>R8G8B8</format>
-                    <width>640</width>
-                    <height>480</height>
-                </image>
-                <clip>
-                    <near>0.05</near>
-                    <far>8.0</far>
-                </clip>
-            </camera>
-            <topic>camera/image_raw</topic>
-            <gz_frame_id>camera_link_optical</gz_frame_id>
+        <sensor name="depth_camera" type="depth_camera">
+        <camera>
+            <horizontal_fov>1.25</horizontal_fov>
+            <image>
+            <width>320</width>
+            <height>240</height>
+            <!-- <format>L16</format> -->
+            </image>
+            <clip>
+            <near>0.1</near>
+            <far>20</far>
+            </clip>
+            <!-- <optical_frame_id>camera_link</optical_frame_id> -->
+            <optical_frame_id>camera_link_optical</optical_frame_id>
+            <!-- <camera_info_topic>camera_info</camera_info_topic> -->
+        </camera>
+        <always_on>1</always_on>
+        <update_rate>20</update_rate>
+        <visualize>true</visualize>
+        <topic>camera_depth</topic>
+        <gz_frame_id>camera_link</gz_frame_id>
+        </sensor>
+        <sensor name="camera" type="camera">
+        <camera>
+            <horizontal_fov>1.25</horizontal_fov>
+            <image>
+            <width>320</width>
+            <height>240</height>
+            <format>R8G8B8</format>
+            </image>
+            <clip>
+            <near>0.1</near>
+            <far>20</far>
+            </clip>
+            <optical_frame_id>camera_link_optical</optical_frame_id>
+            <camera_info_topic>camera_info</camera_info_topic>
+        </camera>
+        <always_on>1</always_on>
+        <update_rate>20</update_rate>
+        <visualize>true</visualize>
+        <topic>camera</topic>
         </sensor>
     </gazebo>

File: description/lidar.xacro (robot description, xacro)
@@ -34,5 +34,5 @@
             <pose relative_to='lidar_frame'> 0 0 0 0 0 0 </pose>
             <update_rate>10</update_rate>
-            <ray>
+            <lidar>
                 <scan>
                     <horizontal>
@@ -48,5 +48,5 @@
                     <resolution>0.01</resolution>
                 </range>
-            </ray>
+            </lidar>
             <topic>scan</topic>
             <gz_frame_id>laser_frame</gz_frame_id>

File: description/robot.urdf.xacro (robot description, xacro)
@@ -2,7 +2,7 @@
 <robot xmlns:xacro="http://www.ros.org/wiki/xacro"  name="robot">
     <xacro:include filename="robot_core.xacro"/>
-    <xacro:include filename="gazebo_control.xacro"/>
+    <xacro:include filename="ros2_control.xacro"/>
     <xacro:include filename="lidar.xacro"/>
-    <!-- <xacro:include filename="camera.xacro"/> -->
-    <xacro:include filename="depth_camera.xacro"/>
+    <xacro:include filename="camera.xacro"/>
+    <!-- <xacro:include filename="depth_camera.xacro"/> -->
 </robot>
